Commit message: obs

File: scout/description/urdf/scout.xacro (robot description, xacro)
@@ -32,5 +32,5 @@
             </geometry>
         </visual>
-        <collision>
+        <collision name = 'base_collision'>
             <origin xyz="0 0 0" rpy="0.0 0.0 0.0"/>
             <geometry>
@@ -198,4 +198,27 @@
             <robotBaseFrame>base_link</robotBaseFrame>
         </plugin>
+    </gazebo>
+    <!-- <gazebo>
+        <plugin name="contact_sensor" filename="libgazebo_ros_bumper.so">
+            <alwaysOn>true</alwaysOn>
+            <updateRate>20</updateRate>
+            <bumperTopicName>bumper</bumperTopicName>
+            <frameName>chasis</frameName>
+        </plugin>
+    </gazebo> -->
+    <gazebo reference="base_link">
+        <sensor name="contact_sensor" type="contact">
+            <always_on>true</always_on>
+            <update_rate>20</update_rate>
+            <contact>
+                <collision>base_link_fixed_joint_lump__base_collision_collision</collision>
+            </contact>
+            <plugin name="bumper" filename="libgazebo_ros_bumper.so">
+                <always_on>true</always_on>
+                    <bumperTopicName>bumper</bumperTopicName>
+                    <frameName>base_link</frameName>
+                <update_rate>20</update_rate>
+            </plugin>
+        </sensor>
     </gazebo>
     <gazebo reference="lidar">

Commit message: 20200417

File: scout/description/urdf/scout.xacro (robot description, xacro)
@@ -218,4 +218,64 @@
                     <bumperTopicName>bumper</bumperTopicName>
                     <frameName>base_link</frameName>
+                <update_rate>20</update_rate>
+            </plugin>
+        </sensor>
+    </gazebo>
+    <gazebo reference="left_front_wheel">
+        <sensor name="contact_sensor1" type="contact">
+            <always_on>true</always_on>
+            <update_rate>20</update_rate>
+            <contact>
+                <collision>left_front_wheel_fixed_joint_lump__base_collision_collision</collision>
+            </contact>
+            <plugin name="bumper" filename="libgazebo_ros_bumper.so">
+                <always_on>true</always_on>
+                    <bumperTopicName>bumper</bumperTopicName>
+                    <frameName>left_front_wheel</frameName>
+                <update_rate>20</update_rate>
+            </plugin>
+        </sensor>
+    </gazebo>
+    <gazebo reference="right_front_wheel">
+        <sensor name="contact_sensor2" type="contact">
+            <always_on>true</always_on>
+            <update_rate>20</update_rate>
+            <contact>
+                <collision>right_front_wheel_fixed_joint_lump__base_collision_collision</collision>
+            </contact>
+            <plugin name="bumper" filename="libgazebo_ros_bumper.so">
+                <always_on>true</always_on>
+                    <bumperTopicName>bumper</bumperTopicName>
+                    <frameName>base_link</frameName>
+                <update_rate>20</update_rate>
+            </plugin>
+        </sensor>
+    </gazebo>
+    <gazebo reference="right_rear_wheel">
+        <sensor name="contact_sensor3" type="contact">
+            <always_on>true</always_on>
+            <update_rate>20</update_rate>
+            <contact>
+                <collision>right_rear_wheel_fixed_joint_lump__base_collision_collision</collision>
+            </contact>
+            <plugin name="bumper" filename="libgazebo_ros_bumper.so">
+                <always_on>true</always_on>
+                    <bumperTopicName>bumper</bumperTopicName>
+                    <frameName>right_rear_wheel</frameName>
+                <update_rate>20</update_rate>
+            </plugin>
+        </sensor>
+    </gazebo>
+    <gazebo reference="left_rear_wheel">
+        <sensor name="contact_sensor4" type="contact">
+            <always_on>true</always_on>
+            <update_rate>20</update_rate>
+            <contact>
+                <collision>left_rear_wheel_fixed_joint_lump__base_collision_collision</collision>
+            </contact>
+            <plugin name="bumper" filename="libgazebo_ros_bumper.so">
+                <always_on>true</always_on>
+                    <bumperTopicName>bumper</bumperTopicName>
+                    <frameName>left_rear_wheel</frameName>
                 <update_rate>20</update_rate>
             </plugin>
@@ -243,5 +303,5 @@
             </scan>
             <range>
-              <min>0.3</min>
+              <min>0.2</min>
               <max>131</max>
               <resolution>0.001</resolution>
@@ -256,5 +316,5 @@
             <topicName>livox/lidar</topicName>
             <frameName>lidar</frameName>
-            <min_range>0.9</min_range>
+            <min_range>0.2</min_range>
             <max_range>130</max_range>
             <gaussianNoise>0.08</gaussianNoise>
