Commit message: 20200511

File: scout/description/urdf/scout_real.xacro (robot description, xacro)
@@ -30,5 +30,5 @@
             <geometry>
                 <!-- <box size="${length} ${width} ${height}"/> -->
-                <mesh filename="package://description/meshes/scout.stl" />
+                <mesh filename="/home/xyw/BUAA/Graduation/src/scout/description/meshes/scout.stl" />
             </geometry>
         </visual>
@@ -60,5 +60,5 @@
             <geometry>
                 <!-- <cylinder radius="${wheelrad}" length="${wheelwid}"/> -->
-                <mesh filename="package://description/meshes/tire.stl" />
+                <mesh filename="/home/xyw/BUAA/Graduation/src/scout/description/meshes/tire.stl" />
             </geometry>
         </visual>
@@ -90,5 +90,5 @@
             <geometry>
                 <!-- <cylinder radius="${wheelrad}" length="${wheelwid}"/> -->
-                <mesh filename="package://description/meshes/tire.stl" />
+                <mesh filename="/home/xyw/BUAA/Graduation/src/scout/description/meshes/tire.stl" />
             </geometry>
         </visual>
@@ -120,5 +120,5 @@
             <geometry>
                 <!-- <cylinder radius="${wheelrad}" length="${wheelwid}"/> -->
-                <mesh filename="package://description/meshes/tire.stl" />
+                <mesh filename="/home/xyw/BUAA/Graduation/src/scout/description/meshes/tire.stl" />
             </geometry>
         </visual>
@@ -150,5 +150,5 @@
             <geometry>
                 <!-- <cylinder radius="${wheelrad}" length="${wheelwid}"/> -->
-                <mesh filename="package://description/meshes/tire.stl" />
+                <mesh filename="/home/xyw/BUAA/Graduation/src/scout/description/meshes/tire.stl" />
             </geometry>
         </visual>

Commit message: 20200522

File: scout/description/urdf/scout_real.xacro (robot description, xacro)
@@ -30,5 +30,5 @@
             <geometry>
                 <!-- <box size="${length} ${width} ${height}"/> -->
-                <mesh filename="/home/xyw/BUAA/Graduation/src/scout/description/meshes/scout.stl" />
+                <mesh filename="/home/xyw/BUAA/Graduation/src/scout/description/meshes/Scout_body.stl" />
             </geometry>
         </visual>
