Commit message: 20200523

File: scout/description/urdf/goal_range.xacro (robot description, xacro)
@@ -1,7 +1,7 @@
 <?xml version="1.0"?>
 <robot name="goal" xmlns:xacro="http://www.ros.org/wiki/xacro">
-  <!-- <link name="world"/>
-  <joint name="fixed" type="continuous">
-    <parent link="world"/>
+  <!-- <link name="set"/>
+  <joint name="fixed" type="fixed">
+    <parent link="set"/>
     <child link="goal"/>
   </joint> -->
@@ -16,7 +16,6 @@
       <origin xyz="0 0 0" rpy="0 0 0"/>
       <geometry>
-        <cylinder radius="0.8" length="500"/>
+        <cylinder radius="0.8" length="3"/>
       </geometry>
-      <material name="green"/>
     </visual>
     <inertial>
@@ -29,3 +28,13 @@
       </inertial>
   </link>
+  <gazebo reference="goal">
+    <visual>
+      <material>
+        <ambient>0 0.5 0 0.01</ambient>
+        <diffuse>0.46 0.46 0.46 0.5</diffuse>
+        <specular>0.5 0.5 0.5 32</specular>
+        <emissive>0.46 0.46 0.46 0.5</emissive>
+      </material>
+    </visual>
+  </gazebo>
 </robot>
