Commit message: 0616

File: scout/description/urdf/goal_final.xacro (robot description, xacro)
@@ -1,6 +1,6 @@
 <?xml version="1.0"?>
-<robot name="goal" xmlns:xacro="http://www.ros.org/wiki/xacro">
+<robot name="range" xmlns:xacro="http://www.ros.org/wiki/xacro">
   <link name="world"/>
-  <joint name="fixed" type="fixed">
+  <!-- <joint name="fixed" type="fixed">
     <parent link="world"/>
     <child link="goal"/>
@@ -27,5 +27,5 @@
         izz="1.0"/>
       </inertial>
-  </link>
+  </link> -->
   <joint name="fixed2" type="fixed">
     <parent link="world"/>
@@ -80,5 +80,5 @@
       </inertial>
   </link>
-  <gazebo reference="goal">
+  <!-- <gazebo reference="goal">
     <visual>
       <material>
@@ -89,5 +89,5 @@
       </material>
     </visual>
-  </gazebo>
+  </gazebo> -->
   <gazebo reference="ori">
     <visual>
